Commit message: implemented IMU sensor broadcaster with imu on hardware

File: description/ros2_control/diffbot.ros2_control.xacro (robot description, xacro)
@@ -7,9 +7,12 @@
         <param name="left_wheel_name">left_wheel_joint</param>
         <param name="right_wheel_name">right_wheel_joint</param>
+        <param name="imu_sensor_name">imu_sensor</param>
         <param name="loop_rate">30</param>
         <param name="device">/dev/ttyACM0</param>
         <param name="baud_rate">921600</param>
         <param name="timeout_ms">1000</param>
-        <param name="enc_counts_per_rev">100</param>
+        <param name="enc_counts_per_rev">792</param>
+        <param name="max_accel_mps">39.24</param>
+        <param name="max_gyro_radps">3141.59</param>
       </hardware>
       <joint name="${prefix}left_wheel_joint">
@@ -23,4 +26,17 @@
         <state_interface name="velocity"/>
       </joint>
+      <sensor name="imu_sensor">
+        <param name="frame_id">imu_link</param>
+        <state_interface name="orientation.x"/>
+        <state_interface name="orientation.y"/>
+        <state_interface name="orientation.z"/>
+        <state_interface name="orientation.w"/>
+        <state_interface name="linear_acceleration.x"/>
+        <state_interface name="linear_acceleration.y"/>
+        <state_interface name="linear_acceleration.z"/>
+        <state_interface name="angular_velocity.x"/>
+        <state_interface name="angular_velocity.y"/>
+        <state_interface name="angular_velocity.z"/>
+      </sensor>
     </ros2_control>
   </xacro:macro>

File: description/urdf/diffbot_description.urdf.xacro (robot description, xacro)
@@ -158,4 +158,26 @@
         </inertial>
       </link>
+    <joint name="${prefix}imu_joint" type="fixed">
+      <parent link="${prefix}base_link"/>
+      <child link="imu_link"/>
+      <origin xyz="0 0 0" rpy="0 0 0"/>
+    </joint>
+    <link name="imu_link">
+      <parent link="${prefix}base_link"/>
+      <visual>
+        <geometry>
+          <box size="0.05 0.05 0.02"/>
+        </geometry>
+      </visual>
+      <collision>
+        <geometry>
+          <box size="0.05 0.05 0.02"/>
+        </geometry>
+      </collision>
+    </link>
+    <sensor name="imu_sensor">
+      <parent link="imu_link"/>
+      <origin xyz="0 0 0" rpy="0 0 0"/>
+    </sensor>
   </xacro:macro>
 </robot>
