Commit message: modified urdf for correct installed IMU orientation. removed mapping of axes in imu_sensor implementation

File: description/urdf/diffbot_description.urdf.xacro (robot description, xacro)
@@ -161,5 +161,5 @@
       <parent link="${prefix}base_link"/>
       <child link="imu_link"/>
-      <origin xyz="0 0 0" rpy="0 0 0"/>
+      <origin xyz="0 0 0" rpy="0 ${PI/2} 0"/>
     </joint>
     <link name="imu_link">
